Commit message: fix: resolve kinematics chain and ros2_control configuration issues

File: cam_auto_adjusting/urdf/robot.urdf.xacro (robot description, xacro)
@@ -3,5 +3,5 @@
   name="cam_auto_adjusting" xmlns:xacro="http://www.ros.org/wiki/xacro">
   <xacro:include filename="robotic_arm.xacro"/>
-  <xacro:include filename="ros2_control_.xacro"/>
+  <!-- ros2_control_.xacro is excluded - use MoveIt config's ros2_control instead -->
   <xacro:include filename="camera.xacro"/>
 </robot>

File: cam_auto_adjusting_config/config/cam_auto_adjusting.ros2_control.xacro (robot description, xacro)
@@ -29,4 +29,11 @@
                 <state_interface name="velocity"/>
             </joint>
+            <joint name="Rotary_01">
+                <command_interface name="position"/>
+                <state_interface name="position">
+                  <param name="initial_value">${initial_positions['Rotary_01']}</param>
+                </state_interface>
+                <state_interface name="velocity"/>
+            </joint>
         </ros2_control>
     </xacro:macro>
