Commit message: fix: adjust interial matrix and mass so the setup does not tilt

File: cam_auto_adjusting/urdf/robotic_arm.xacro (robot description, xacro)
@@ -55,6 +55,6 @@
     <inertial>
       <origin xyz="0 0 0" rpy="0 0 0"/>
-      <mass value="1.0"/>
-      <inertia ixx="0.01" ixy="0.0" ixz="0.0" iyy="0.01" iyz="0.0" izz="0.01"/>
+      <mass value="0.1"/>
+      <inertia ixx="0.0001" ixy="0.0" ixz="0.0" iyy="0.0001" iyz="0.0" izz="0.0001"/>
     </inertial>
     <visual>

Commit message: fix: adjust interial tag for Object

File: cam_auto_adjusting/urdf/robotic_arm.xacro (robot description, xacro)
@@ -25,7 +25,7 @@
   <link name="Rotary">
     <inertial>
-      <origin xyz="2.77555756156289E-17 -5.55111512312578E-17 0.038" rpy="0 0 0" />
-      <mass value="0.251327412287183" />
-      <inertia ixx="0.000223513845327402" ixy="9.45007218889529E-37" ixz="6.54556654792952E-20" iyy="0.000223513845327402" iyz="4.9904894759554E-21" izz="0.000412176956150981" />
+      <origin xyz="0 0 0.038" rpy="0 0 0" />
+      <mass value="0.4" />
+      <inertia ixx="0.000356" ixy="0.0" ixz="0.0" iyy="0.000356" iyz="0.0" izz="0.000656" />
     </inertial>
     <visual>
@@ -55,11 +55,12 @@
     <inertial>
       <origin xyz="0 0 0" rpy="0 0 0"/>
-      <mass value="0.1"/>
-      <inertia ixx="0.0001" ixy="0.0" ixz="0.0" iyy="0.0001" iyz="0.0" izz="0.0001"/>
+      <mass value="0.3"/>
+      <inertia ixx="0.0003" ixy="0.0" ixz="0.0" iyy="0.0003" iyz="0.0" izz="0.0003"/>
     </inertial>
     <visual>
       <origin xyz="0 0 0" rpy="0 0 0"/>
       <geometry>
-        <mesh filename="package://cam_auto_adjusting/meshes/drill_bit_two.dae" scale="0.7 0.7 0.7"/>
+        <mesh filename="package://cam_auto_adjusting/meshes/drill_bit_two.dae" scale="0.5 0.5 0.5"/>
+        <!-- <mesh filename="package://cam_auto_adjusting/meshes/drill_bit_one.obj" scale="1 1 1"/> -->
       </geometry>
     </visual>
@@ -67,5 +68,6 @@
       <origin xyz="0 0 0" rpy="0 0 0"/>
       <geometry>
-        <mesh filename="package://cam_auto_adjusting/meshes/drill_bit_two.dae" scale="0.7 0.7 0.7"/>
+        <mesh filename="package://cam_auto_adjusting/meshes/drill_bit_two.dae" scale="0.5 0.5 0.5"/>
+        <!-- <mesh filename="package://cam_auto_adjusting/meshes/drill_bit_one.obj" scale="1 1 1"/> -->
       </geometry>
     </collision>
